File: hardware/V0.0.1/dual_wbo.brd (EAGLE design)
At the start: 100 x 80 mm, 65 parts, among them IC1 CJ125_QFP32, IC3 AT90CAN128, IC4 CJ125_QFP32, IC5 TJA1051T, IC6 AVR-JTAG, IC7 REF50XX, Q1 16MHz

Commit message: -> dac name corrected -> dac datasheet added
Parts:
- added C26, C29: 100nF, rcl:C0603
- added C27, C30: 10µF, Heinrich:SMC_C
- added C28: 470nF, rcl:C0603
- added IC2: TLS115B0EJXUMA1, Heinrich:SOIC127P600X170-9N
- C19, C20: value 100nF -> 470nF
- moved IC7 8.35 mm to (21.0, 15.2), turned to 180 degrees
Connections:
- new net 5V_REF: C26.1, IC2.5, IC7.6
- net +UBAT: now also C27.+, C28.1, C30.+, IC2.7, IC2.8
- net AGND: now also C26.2, C29.2
- net AREF: now also C29.1, IC2.1; no longer IC7.6
- net GND: now also C27.-, C28.2, C30.-, IC2.3, IC2.9
Routing:
- net 5V_REF: track 0.00 -> 10.6 mm
- net +UBAT: track 0.00 -> 9.34 mm
- net AREF: track 0.00 -> 7.94 mm

Commit message: some changes
Parts:
- moved C13 5.46 mm to (54.0, 36.2), turned to 180 degrees
- moved C12 4.84 mm to (48.9, 36.2), turned to 180 degrees
- moved Q1 0.90 mm to (51.4, 40.0)
Connections:
- net AGND: now also C8.2
- net GND: no longer C8.2
Routing:
- net XTAL1: track 8.68 -> 10.2 mm
Changed lines of the file:
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@@
 <attribute name="SPICEPREFIX" value="C" x="85.09" y="52.07" size="1.778" layer="27" rot="R270" display="off"/>
 </element>
-<element name="C12" library="rcl" library_urn="urn:adsk.eagle:library:334" package="C0603" package3d_urn="urn:adsk.eagle:package:23616/2" value="18pF" x="46.99" y="40.64" smashed="yes" rot="R90">
-<attribute name="NAME" x="46.355" y="40.005" size="1.27" layer="25" rot="R90"/>
-<attribute name="SPICEPREFIX" value="C" x="46.99" y="40.64" size="1.778" layer="27" rot="R90" display="off"/>
-</element>
-<element name="C13" library="rcl" library_urn="urn:adsk.eagle:library:334" package="C0603" package3d_urn="urn:adsk.eagle:package:23616/2" value="18pF" x="57.15" y="40.64" smashed="yes" rot="R90">
-<attribute name="NAME" x="56.515" y="40.005" size="1.27" layer="25" rot="R90"/>
-<attribute name="SPICEPREFIX" value="C" x="57.15" y="40.64" size="1.778" layer="27" rot="R90" display="off"/>
+<element name="C12" library="rcl" library_urn="urn:adsk.eagle:library:334" package="C0603" package3d_urn="urn:adsk.eagle:package:23616/2" value="18pF" x="48.895" y="36.195" smashed="yes" rot="R180">
+<attribute name="NAME" x="49.53" y="35.56" size="1.27" layer="25" rot="R180"/>
+<attribute name="SPICEPREFIX" value="C" x="48.895" y="36.195" size="1.778" layer="27" rot="R180" display="off"/>
+</element>
+<element name="C13" library="rcl" library_urn="urn:adsk.eagle:library:334" package="C0603" package3d_urn="urn:adsk.eagle:package:23616/2" value="18pF" x="53.975" y="36.195" smashed="yes" rot="R180">
+<attribute name="NAME" x="54.61" y="35.56" size="1.27" layer="25" rot="R180"/>
+<attribute name="SPICEPREFIX" value="C" x="53.975" y="36.195" size="1.778" layer="27" rot="R180" display="off"/>
 </element>
 <element name="C14" library="rcl" library_urn="urn:adsk.eagle:library:334" package="C0603" package3d_urn="urn:adsk.eagle:package:23616/2" value="100nF" x="85.09" y="59.69" smashed="yes" rot="R270">
@@
 <attribute name="NAME" x="85.725" y="66.675" size="1.27" layer="25" rot="R270"/>
 </element>
-<element name="Q1" library="Heinrich" package="ABM3" value="16MHz" x="52.07" y="40.64" smashed="yes" rot="R180">
-<attribute name="ARROW_PART_NUMBER" value="ABM3-8.000MHZ-D2Y-T" x="52.07" y="40.64" size="1.778" layer="27" rot="R180" display="off"/>
-<attribute name="ARROW_PRICE-STOCK" value="https://www.arrow.com/en/products/abm3-8.000mhz-d2y-t/abracon?region=nac" x="52.07" y="40.64" size="1.778" layer="27" rot="R180" display="off"/>
-<attribute name="DESCRIPTION" value="Abracon 6 MHz, 8 MHz Crystal +/-20 ppm, +/-30 ppm 2-SMD, HC49/US, No Lead" x="52.07" y="40.64" size="1.778" layer="27" rot="R180" display="off"/>
-<attribute name="HEIGHT" value="1mm" x="52.07" y="40.64" size="1.778" layer="27" rot="R180" display="off"/>
-<attribute name="MANUFACTURER_NAME" value="ABRACON" x="52.07" y="40.64" size="1.778" layer="27" rot="R180" display="off"/>
-<attribute name="MANUFACTURER_PART_NUMBER" value="ABM3-8.000MHZ-D2Y-T" x="52.07" y="40.64" size="1.778" layer="27" rot="R180" display="off"/>
-<attribute name="MOUSER_PART_NUMBER" value="815-ABM3-8-D2Y-T" x="52.07" y="40.64" size="1.778" layer="27" rot="R180" display="off"/>
-<attribute name="MOUSER_PRICE-STOCK" value="https://www.mouser.co.uk/ProductDetail/ABRACON/ABM3-8000MHZ-D2Y-T?qs=ihRgKfnEsN4giUXjc3yS1g%3D%3D" x="52.07" y="40.64" size="1.778" layer="27" rot="R180" display="off"/>
-<attribute name="NAME" x="53.34" y="44.45" size="1.27" layer="25" rot="R180" align="center"/>
-</element>
 <element name="R1" library="rcl" library_urn="urn:adsk.eagle:library:334" package="R0603" package3d_urn="urn:adsk.eagle:package:23555/2" value="10k" x="34.925" y="61.595" smashed="yes">
 <attribute name="NAME" x="34.29" y="62.23" size="1.27" layer="25"/>
@@
 </element>
 <element name="C30" library="Heinrich" package="SMC_C" value="10µF" x="30.48" y="3.175"/>
+<element name="Q1" library="Heinrich" package="ABM3" value="16MHz" x="51.435" y="40.005" rot="R180">
+<attribute name="ARROW_PART_NUMBER" value="ABM3-8.000MHZ-D2Y-T" x="51.435" y="40.005" size="1.778" layer="27" rot="R180" display="off"/>
+<attribute name="ARROW_PRICE-STOCK" value="https://www.arrow.com/en/products/abm3-8.000mhz-d2y-t/abracon?region=nac" x="51.435" y="40.005" size="1.778" layer="27" rot="R180" display="off"/>
+<attribute name="DESCRIPTION" value="Abracon 6 MHz, 8 MHz Crystal +/-20 ppm, +/-30 ppm 2-SMD, HC49/US, No Lead" x="51.435" y="40.005" size="1.778" layer="27" rot="R180" display="off"/>
+<attribute name="HEIGHT" value="1mm" x="51.435" y="40.005" size="1.778" layer="27" rot="R180" display="off"/>
+<attribute name="MANUFACTURER_NAME" value="ABRACON" x="51.435" y="40.005" size="1.778" layer="27" rot="R180" display="off"/>
+<attribute name="MANUFACTURER_PART_NUMBER" value="ABM3-8.000MHZ-D2Y-T" x="51.435" y="40.005" size="1.778" layer="27" rot="R180" display="off"/>
+<attribute name="MOUSER_PART_NUMBER" value="815-ABM3-8-D2Y-T" x="51.435" y="40.005" size="1.778" layer="27" rot="R180" display="off"/>
+<attribute name="MOUSER_PRICE-STOCK" value="https://www.mouser.co.uk/ProductDetail/ABRACON/ABM3-8000MHZ-D2Y-T?qs=ihRgKfnEsN4giUXjc3yS1g%3D%3D" x="51.435" y="40.005" size="1.778" layer="27" rot="R180" display="off"/>
+</element>
 </elements>
 <signals>
@@
 <contactref element="C1" pad="2"/>
 <contactref element="C3" pad="2"/>
-<contactref element="C8" pad="2"/>
 <contactref element="C7" pad="2"/>
 <contactref element="IC4" pad="29"/>
@@
 <signal name="XTAL1">
 <contactref element="IC3" pad="23"/>
+<contactref element="C12" pad="1"/>
 <contactref element="Q1" pad="2"/>
-<contactref element="C12" pad="1"/>
-<wire x1="50.8889" y1="45.5803" x2="50.8889" y2="41.5089" width="0.254" layer="1"/>
-<wire x1="50.8889" y1="41.5089" x2="50.02" y2="40.64" width="0.254" layer="1"/>
-<wire x1="50.02" y1="40.64" x2="48.26" y2="40.64" width="0.254" layer="1"/>
-<wire x1="48.26" y1="40.64" x2="47.41" y2="39.79" width="0.254" layer="1"/>
-<wire x1="47.41" y1="39.79" x2="46.99" y2="39.79" width="0.254" layer="1"/>
+<wire x1="50.8889" y1="45.5803" x2="50.8889" y2="41.5089" width="0.1524" layer="1"/>
+<wire x1="50.8889" y1="41.5089" x2="49.4575" y2="40.0775" width="0.1524" layer="1"/>
+<wire x1="49.4575" y1="40.0775" x2="49.385" y2="40.005" width="0.1524" layer="1"/>
+<wire x1="49.745" y1="36.195" x2="49.745" y2="39.79" width="0.1524" layer="1"/>
+<wire x1="49.745" y1="39.79" x2="49.4575" y2="40.0775" width="0.1524" layer="1"/>
 </signal>
 <signal name="XTAL2">
 <contactref element="IC3" pad="24"/>
+<contactref element="C13" pad="2"/>
 <contactref element="Q1" pad="1"/>
-<contactref element="C13" pad="2"/>
-<wire x1="51.6763" y1="45.5803" x2="51.6763" y2="41.0337" width="0.254" layer="1"/>
-<wire x1="51.6763" y1="41.0337" x2="52.07" y2="40.64" width="0.254" layer="1"/>
-<wire x1="52.07" y1="40.64" x2="54.12" y2="40.64" width="0.254" layer="1"/>
-<wire x1="56.3" y1="40.64" x2="57.15" y2="41.49" width="0.254" layer="1"/>
-<wire x1="54.12" y1="40.64" x2="56.3" y2="40.64" width="0.254" layer="1"/>
+<wire x1="51.6763" y1="45.5803" x2="51.6763" y2="41.8137" width="0.1524" layer="1"/>
+<wire x1="51.6763" y1="41.8137" x2="53.4125" y2="40.0775" width="0.1524" layer="1"/>
+<wire x1="53.4125" y1="40.0775" x2="53.485" y2="40.005" width="0.1524" layer="1"/>
+<wire x1="53.125" y1="36.195" x2="53.125" y2="39.79" width="0.1524" layer="1"/>
+<wire x1="53.125" y1="39.79" x2="53.4125" y2="40.0775" width="0.1524" layer="1"/>
 </signal>
 <signal name="!RESET">
@@
 <contactref element="C26" pad="2"/>
 <contactref element="C29" pad="2"/>
+<contactref element="C8" pad="2"/>
+<wire x1="46.9519" y1="61.0997" x2="80.01" y2="74.08" width="0" layer="19" extent="1-1"/>
 <wire x1="22.716828125" y1="60.112515625" x2="46.9519" y2="61.0997" width="0" layer="19" extent="1-1"/>
 <wire x1="9.105" y1="53.975" x2="22.716828125" y2="60.112515625" width="0" layer="19" extent="1-1"/>
