File: hardware/V0.0.1/dual_wbo.sch (EAGLE design)
At the start: 65 parts, among them IC1 CJ125_QFP32, IC3 AT90CAN128, IC4 CJ125_QFP32, IC5 TJA1051T, IC6 AVR-JTAG, IC7 REF50XX, Q1 16MHz

Commit message: -> dac name corrected -> dac datasheet added
Parts:
- added C26, C29: 100nF, rcl:C-EUC0603
- added C27, C30: 10µF, Heinrich:CAP_TANTALUMSMCC
- added C28: 470nF, rcl:C-EUC0603
- added IC2: TLS115B0EJXUMA1, Heinrich:TLS115B0EJXUMA1
- C19, C20: value 100nF -> 470nF
Connections:
- new net 5V_REF: C26.1, IC2.ADJ, IC7.VOUT
- net +UBAT: now also C27.+, C28.1, C30.+, IC2.EN, IC2.IN
- net AGND: now also C26.2, C29.2
- net AREF: now also C29.1, IC2.OUT; no longer IC7.VOUT
- net GND: now also C27.-, C28.2, C30.-, IC2.GND
Other:
- moved on the sheet: C17, C20, D2, IC7, R25, R26

Commit message: some changes
Connections:
- net AGND: now also C8.2
- net GND: no longer C8.2
Other:
- moved on the sheet: D1
